File: Skull Candy Lamp.brd (EAGLE design)
At the start: 96.2 x 43 mm, 22 parts, among them IC1 74HCT125D, J2 SERIAL, U1 M5STAMP PICO

Commit message: cosmetic updates
Parts:
- moved J2 2.00 mm to (54.6, 14.0), turned to 0 degrees
- moved C5 0.38 mm to (67.8, 27.9)
- renumbered S1 to FLASH
Routing:
- net GND: track 25.9 -> 21.7 mm
- net RX: track 42.3 -> 41.3 mm
- net DI$8: track 21.3 -> 20.5 mm
- net TX: track 33.0 -> 32.3 mm
- net VCC: track 232.7 -> 232.5 mm, vias 2 -> 1
